File: Mini-Speaker_Amplifier/Mini-Speaker_Amplifier.sch (KiCad schematic (older format))
At the start: 13 parts, among them J1 AudioJack2, J2 Conn_02x05, U1 LM386

Commit message: Added reverse protection diode Make grid raster 0.5080
Parts:
- added D?: 1N5817, Diode_THT:D_DO-41_SOD81_P10.16mm_Horizontal, symbol Diode:1N5817
Connections:
- wire segments 44 -> 45
Changed lines of the file:
@@
 EESchema Schematic File Version 4
-LIBS:Mini-Speaker_Amplifier-cache
 EELAYER 30 0
 EELAYER END
@@
 Wire Wire Line
 	5300 4750 5800 4750
-Connection ~ 5800 4750
 Connection ~ 5300 4850
 Connection ~ 5800 4850
@@
 	1    0    0    -1
 $EndComp
-Wire Wire Line
-	7150 4550 7150 4750
-Connection ~ 7150 4750
-Wire Wire Line
-	7150 4750 7150 4800
-Wire Wire Line
-	5800 4750 7150 4750
-$Comp
-L clacktronics_schematic_logo:LOGO #G1
+$Comp
+L Mini-Speaker_Amplifier-rescue:LOGO-clacktronics_schematic_logo #G1
 U 1 1 5D2D236A
 P 8450 6800
@@
 	1    0    0    -1
 $EndComp
+Wire Wire Line
+	7150 4550 7150 4750
+$Comp
+L Diode:1N5817 D?
+U 1 1 661F2DF8
+P 6400 4750
+F 0 "D?" H 6400 4533 50  0000 C CNN
+F 1 "1N5817" H 6400 4624 50  0000 C CNN
+F 2 "Diode_THT:D_DO-41_SOD81_P10.16mm_Horizontal" H 6400 4575 50  0001 C CNN
+F 3 "http://www.vishay.com/docs/88525/1n5817.pdf" H 6400 4750 50  0001 C CNN
+	1    6400 4750
+	-1   0    0    1
+$EndComp
+Wire Wire Line
+	6250 4750 5800 4750
+Connection ~ 5800 4750
+Wire Wire Line
+	6550 4750 7150 4750
+Connection ~ 7150 4750
+Wire Wire Line
+	7150 4750 7150 4800
 $EndSCHEMATC
